File: pcb/main_kb/matrix.kicad_sch (KiCad schematic)
At the start: 126 parts, among them SW1 `~, SW10 9, SW11 0, SW12 -_, SW13 =+, SW14 Backspace, SW15 tab, SW16 q, SW17 w, SW18 e, SW19 r, SW2 1, SW20 t, SW21 y, SW22 u, SW23 i, SW24 o, SW25 p, SW26 [{, SW27 ]}, SW28 \ |, SW29 control, SW3 2, SW30 a, SW31 s, SW32 d, SW33 f, SW34 g, SW35 h, SW36 j, SW37 k, SW38 l, SW39 ; :, SW4 3, SW40 esc, SW41 ' ", SW42 enter, SW43 shift, SW44 z, SW45 x, SW46 c, SW47 v, SW48 b, SW49 n, SW5 4, SW50 m, SW51 ,<, SW52 .>, SW53 /?, SW54 rshift, SW55 ↑, SW57 control, SW58 alt, SW59 cmd, SW6 5, SW63 space, SW67 fn, SW68 ←, SW69 ↓, SW7 6, SW70 →, SW8 7, SW9 8

Commit message: Fixed type C Mess
Connections:
- net col 6: now also SW63.2
Changed lines of the file:
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@@
   (junction (at 74.93 86.36) (diameter 0) (color 0 0 0 0)
   )
+  (junction (at 142.24 86.36) (diameter 0) (color 0 0 0 0)
+  )
   (junction (at 195.58 60.96) (diameter 0) (color 0 0 0 0)
   )
@@
     (stroke (width 0) (type default))
   )
+  (wire (pts (xy 142.24 86.36) (xy 142.24 100.33))
+    (stroke (width 0) (type default))
+  )

Commit message: Changed layout, added layout diagram
Parts:
- removed D41, D55: 1N914, Diode_THT:D_DO-35_SOD27_P7.62mm_Horizontal, symbol Diode:1N914
- removed SW54: rshift, symbol Switch:SW_Push
- added D1: 1N914, Diode_THT:D_DO-35_SOD27_P7.62mm_Horizontal, symbol Diode:1N914
- added S2: 6.25u Space, PCM_marbastlib-mx:STAB_MX_P_6.25u, symbol marbastlib-mx:MX_stab
- added S3: 7u Space, PCM_marbastlib-mx:STAB_MX_P_6.25u, symbol marbastlib-mx:MX_stab
- added S4: Shift, PCM_marbastlib-mx:STAB_MX_P_6.25u, symbol marbastlib-mx:MX_stab
Connections:
- net col 10: now also SW40.2; no longer SW67.2
- net col 13: no longer SW40.2
- net row 4: now also D1.1 (K)
- net at SW40.1: now also D1.2 (A)
Other:
- title: (none) ->  Keyflex QWERTY [P.O.D] (C) Rithul K
